File: 001 PCB/TheENDGAME2024_SILKSCREEN.kicad_pcb (KiCad board)
At the start: 2 copper layers, 219 x 96.1 mm, 93 parts, among them J1 B+, J2 B-, SW1 SW_SPDT, SW10 SW_Push, SW11 SW_Push, SW12 SW_Push, SW13 SW_Push, SW14 SW_Push, SW15 SW_Push, SW16 SW_Push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

Commit message: fixed positioning of hole
Parts:
- moved REF** 1.52 mm to (255.4, 146.3)
